File: RFM98LPC824/LPC824_RFM9x.kicad_pcb (KiCad board)
At the start: 2 copper layers, 38.9 x 16.5 mm, 18 parts, among them J2 Conn_01x03, J3 Conn_01x06, J4 Conn_01x06, U1 LPC824M201JDH20, U2 RFM92/95/96/97/98, U3 AT25_EEPROM

Commit message: no comment
Other:
- board text added: "FarmEye Soil Temperature Probe"
Changed lines of the file:
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@@
     (links 44)
     (no_connects 1)
-    (area 140.894999 97.714999 179.907001 114.375001)
+    (area 137.592381 96.127 192.635 121.826001)
     (thickness 1.6)
-    (drawings 30)
+    (drawings 31)
     (tracks 214)
     (zones 0)
@@
       (xy -0.117902 -2.924174) (xy -0.057389 -2.933563) (xy -0.006332 -2.910978)) (layer B.Mask) (width 0.01))
   )
+  (gr_text "FarmEye \nSoil Temperature \nProbe" (at 165.862 112.014) (layer F.SilkS)
+    (effects (font (size 0.5 0.5) (thickness 0.1)))
+  )
   (gr_text FARMEYE (at 177.8 108.712 90) (layer B.SilkS)
